File: projects/route-test/route-test.kicad_pcb (KiCad board)
At the start: 2 copper layers, 0 parts

Commit message: route-test: footprints synced from schematic and placed via IPC, 30x20mm outline
Co-Authored-By: Claude Opus 5.5 <noreply@anthropic.com>
Parts:
- added J1: Conn_01x03, Connector_PinHeader_2.54mm:PinHeader_1x03_P2.54mm_Vertical, F.Cu at (104.0, 107.5)
- added R1: 10k, Resistor_SMD:R_0805_2012Metric, F.Cu at (118.0, 106.0)
- added R2: 10k, Resistor_SMD:R_0805_2012Metric, F.Cu at (118.0, 114.0)
Other:
- board outline added: 30 x 20 mm
