File: projects/route-test/route-test.kicad_sch (KiCad schematic)
At the start: 0 parts

Commit message: route-test: voltage divider schematic (ERC 0 violations)
Co-Authored-By: Claude Opus 5.5 <noreply@anthropic.com>
Parts:
- added J1: Conn_01x03, Connector_PinHeader_2.54mm:PinHeader_1x03_P2.54mm_Vertical, symbol Connector_Generic:Conn_01x03
- added R1, R2: 10k, Resistor_SMD:R_0805_2012Metric, symbol Device:R
Connections:
- new net GND: J1.3 (Pin_3), R2.2
- new net VIN: J1.1 (Pin_1), R1.1
- new net VOUT: J1.2 (Pin_2), R1.2, R2.1

Commit message: route-test: R1/R2 footprints to R_Axial_DIN0207 THT (ERC 0 violations)
Co-Authored-By: Claude Opus 5.5 <noreply@anthropic.com>
Parts:
- R1, R2: footprint Resistor_SMD:R_0805_2012Metric -> Resistor_THT:R_Axial_DIN0207_L6.3mm_D2.5mm_P7.62mm_Horizontal
Changed lines of the file:
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@@
 			)
 		)
-		(property "Footprint" "Resistor_SMD:R_0805_2012Metric"
+		(property "Footprint" "Resistor_THT:R_Axial_DIN0207_L6.3mm_D2.5mm_P7.62mm_Horizontal"
 			(at 130.81 95.25 0)
 			(hide yes)
@@
 			)
 		)
-		(property "Footprint" "Resistor_SMD:R_0805_2012Metric"
+		(property "Footprint" "Resistor_THT:R_Axial_DIN0207_L6.3mm_D2.5mm_P7.62mm_Horizontal"
 			(at 130.81 110.49 0)
 			(hide yes)
