File: projects/cm-carrier/cm.kicad_sch (KiCad schematic)
At the start: 5 parts, among them J2 DEBUG_UART, SW1 PWR_BUT

Commit message: cm-carrier: USB hub sheet (USB2514B, 3 switched ports: Type-C + 2x XA); open-issues list
Co-Authored-By: Claude Opus 5.5 <noreply@anthropic.com>
Connections:
- net HUB_RESET_N: now reaches Module1.100 (CAM_GPIO1)
- no-connect marks 100 -> 99
Changed lines of the file:
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@@
 	(paper "A2")
-	(no_connect
-		(at 119.38 279.4)
-	)
 	(no_connect
 		(at 119.38 172.72)
@@
 		)
 	)
+	(wire
+		(pts
+			(xy 119.38 279.4)
+			(xy 116.84 279.4)
+		)
+	)
 	(label "GND"
 		(at 180.34 154.94 0)
@@
 		)
 	)
+	(global_label "HUB_RESET_N"
+		(shape input)
+		(at 116.84 279.4 180)
+		(effects
+			(font
+				(size 1.27 1.27)
+			)
+			(justify right)
+		)
+	)

Commit message: cm-carrier: LTE sheet (EC25-J Mini PCIe, nanoSIM, open-drain PERST#/W_DISABLE#); move LTE control to GPIO22/23
Co-Authored-By: Claude Opus 5.5 <noreply@anthropic.com>
Connections:
- net LTE_RESET: now reaches Module1.46 (GPIO22)
- net LTE_AIRPLANE: now reaches Module1.47 (GPIO23)
- net LTE_RESET_N: no longer names the net of Module1.30 (GPIO6)
- net LTE_W_DISABLE_N: no longer names the net of Module1.37 (GPIO7)
Changed lines of the file:
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@@
-	)
-	(no_connect
-		(at 119.38 210.82)
-	)
-	(no_connect
-		(at 180.34 213.36)
 	)
 	(no_connect
@@
 	(no_connect
 		(at 330.2 269.24)
+	)
+	(no_connect
+		(at 119.38 190.5)
+	)
+	(no_connect
+		(at 180.34 200.66)
 	)
 	(wire
@@
 	(wire
 		(pts
-			(xy 119.38 190.5)
-			(xy 116.84 190.5)
-		)
-	)
-	(wire
-		(pts
-			(xy 180.34 200.66)
-			(xy 182.88 200.66)
-		)
-	)
-	(wire
-		(pts
 			(xy 180.34 190.5)
 			(xy 182.88 190.5)
@@
 		)
 	)
+	(wire
+		(pts
+			(xy 119.38 210.82)
+			(xy 116.84 210.82)
+		)
+	)
+	(wire
+		(pts
+			(xy 180.34 213.36)
+			(xy 182.88 213.36)
+		)
+	)
 	(label "GND"
 		(at 180.34 154.94 0)
@@
 		)
 	)
-	(global_label "LTE_RESET_N"
-		(shape input)
-		(at 116.84 190.5 180)
-		(effects
-			(font
-				(size 1.27 1.27)
-			)
-			(justify right)
-		)
-	)
-	(global_label "LTE_W_DISABLE_N"
-		(shape input)
-		(at 182.88 200.66 0)
-		(effects
-			(font
-				(size 1.27 1.27)
-			)
-			(justify left)
-		)
-	)
 	(global_label "LTE_3V3_PG"
 		(shape input)
@@
 		)
 	)
+	(global_label "LTE_RESET"
+		(shape input)
+		(at 116.84 210.82 180)
+		(effects
+			(font
+				(size 1.27 1.27)
+			)
+			(justify right)
+		)
+	)
+	(global_label "LTE_AIRPLANE"
+		(shape input)
+		(at 182.88 213.36 0)
+		(effects
+			(font
+				(size 1.27 1.27)
+			)
+			(justify left)
+		)
+	)
